File: hardware/SMART_PJU.brd (EAGLE design)
At the start: 148.2 x 60 mm, 73 parts, among them IC1 DS3231/SO, IC10 ACS712ELCTR-05B-T, IC2 FOD817BSD, IC20 LM358_SOIC, K1 SSR, Q1 PNP, Q2 NMOSFET, Q3 NMOSFET, T20 ZMPT101B, U1 RA-01H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

Commit message: update hardware
Parts:
- removed D1: MBR0520LT1G, Diode:SODFL3718X115
Connections:
- net 5V: now also AMS1117.3, C3.1; no longer D1.2
- net VIN: no longer AMS1117.3, C3.1, D1.1
Routing:
- net VIN: track 81.5 -> 67.0 mm
- net 5V: track 146.1 -> 153.7 mm
Changed lines of the file:
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@@
 <drawing>
 <settings>
-<setting alwaysvectorfont="yes"/>
+<setting alwaysvectorfont="no"/>
 <setting verticaltext="up"/>
 </settings>
@@
 <attribute name="VALUE" x="92.098" y="-5.57" size="0.6" layer="28" ratio="13" rot="MR90" align="top-left"/>
 </element>
-<element name="D1" library="Diode" library_urn="urn:adsk.eagle:library:16378169" package="SODFL3718X115" package3d_urn="urn:adsk.eagle:package:9427153/2" value="MBR0520LT1G" x="86.258" y="-17.071" smashed="yes" rot="R270">
-<attribute name="CATEGORY" value="Diode" x="86.258" y="-17.071" size="0.3048" layer="27" rot="R270" display="off"/>
-<attribute name="DESCRIPTION" value="DIODE SCHOTTKY 20V 500MA SOD123" x="86.258" y="-17.071" size="0.3048" layer="27" rot="R270" display="off"/>
-<attribute name="FORWARD_CURRENT" value="" x="86.258" y="-17.071" size="0.3048" layer="27" rot="R270" display="off"/>
-<attribute name="MANUFACTURER" value="ON Semiconductor" x="86.258" y="-17.071" size="0.3048" layer="27" rot="R270" display="off"/>
-<attribute name="MPN" value="MBR0520LT1G" x="86.258" y="-17.071" size="0.3048" layer="27" rot="R270" display="off"/>
-<attribute name="NAME" x="84.4876" y="-18.071" size="0.6" layer="25" ratio="13" rot="R270" align="bottom-center"/>
-<attribute name="OPERATING_TEMP" value="" x="86.258" y="-17.071" size="0.3048" layer="27" rot="R270" display="off"/>
-<attribute name="PART_STATUS" value="" x="86.258" y="-17.071" size="0.3048" layer="27" rot="R270" display="off"/>
-<attribute name="REVERSE_VOLTAGE" value="" x="86.258" y="-17.071" size="0.3048" layer="27" rot="R270" display="off"/>
-<attribute name="ROHS_COMPLIANT" value="" x="86.258" y="-17.071" size="0.3048" layer="27" rot="R270" display="off"/>
-<attribute name="SERIES" value="" x="86.258" y="-17.071" size="0.3048" layer="27" rot="R270" display="off"/>
-<attribute name="SUB-CATEGORY" value="Schottky" x="86.258" y="-17.071" size="0.3048" layer="27" rot="R270" display="off"/>
-<attribute name="THERMALLOSS" value="" x="86.258" y="-17.071" size="0.3048" layer="27" rot="R270" display="off"/>
-<attribute name="TYPE" value="" x="86.258" y="-17.071" size="0.3048" layer="27" rot="R270" display="off"/>
-<attribute name="VALUE" x="84.6284" y="-17.071" size="0.6" layer="27" ratio="13" rot="R270" align="top-center"/>
-<attribute name="ZENER_VOLTAGE" value="" x="86.258" y="-17.071" size="0.3048" layer="27" rot="R270" display="off"/>
-</element>
 <element name="C3" library="Capacitor" library_urn="urn:adsk.eagle:library:16290819" package="CAPC1608X85" package3d_urn="urn:adsk.eagle:package:16290898/2" value="10µ" x="82.816" y="-19.589" smashed="yes" rot="R270">
 <attribute name="CATEGORY" value="Capacitor" x="82.816" y="-19.589" size="0.3048" layer="27" rot="R270" display="off"/>
@@
 <contactref element="JP1" pad="1"/>
 <contactref element="JP1" pad="10"/>
-<contactref element="D1" pad="2"/>
-<wire x1="86.258" y1="-18.6714" x2="86.258" y2="-21.492" width="0.508" layer="1"/>
 <wire x1="86.258" y1="-21.492" x2="85.92" y2="-21.83" width="0.508" layer="1"/>
 <wire x1="85.92" y1="-21.83" x2="85.92" y2="-22.03" width="0.508" layer="1"/>
@@
 <via x="9.4662625" y="20.453" extent="1-16" drill="0.65"/>
 <wire x1="-3.1" y1="22.5" x2="-1.053" y2="20.453" width="0.508" layer="16"/>
-<wire x1="10.24" y1="-17.94" x2="85.92" y2="-21.83" width="0" layer="19" extent="1-1"/>
+<contactref element="AMS1117" pad="3"/>
+<contactref element="C3" pad="1"/>
+<wire x1="82.872" y1="-15.64" x2="82.85158125" y2="-16.79738125" width="0.508" layer="1"/>
+<wire x1="82.816" y1="-18.8144" x2="82.85158125" y2="-16.79738125" width="0.508" layer="1"/>
+<wire x1="84" y1="-15.64" x2="86.0886" y2="-15.64" width="0.508" layer="1"/>
+<wire x1="82.85158125" y1="-16.79738125" x2="83.52448125" y2="-16.12448125" width="0.508" layer="1"/>
+<wire x1="83.52448125" y1="-16.12448125" x2="84" y2="-15.6489625" width="0.508" layer="1"/>
+<wire x1="84" y1="-15.6489625" x2="84" y2="-15.64" width="0.508" layer="1"/>
+<wire x1="83.3" y1="-15.64" x2="82.872" y2="-15.64" width="0.508" layer="1"/>
+<wire x1="83.3" y1="-15.64" x2="84" y2="-15.64" width="0.508" layer="1"/>
+<wire x1="83.3" y1="-15.64" x2="83.9910375" y2="-15.64" width="0.1524" layer="1"/>
+<wire x1="83.52448125" y1="-16.12448125" x2="83.3" y2="-15.9" width="0.1524" layer="1"/>
+<wire x1="83.3" y1="-15.9" x2="83.3" y2="-15.64" width="0.1524" layer="1"/>
+<wire x1="82.872" y1="-15.64" x2="83.9910375" y2="-15.64" width="0.4064" layer="1"/>
+<wire x1="83.9910375" y1="-15.64" x2="84" y2="-15.6489625" width="0.4064" layer="1"/>
+<wire x1="85.92" y1="-21.83" x2="82.816" y2="-18.8144" width="0" layer="19" extent="1-1"/>
+<wire x1="10.24" y1="-17.94" x2="82.816" y2="-18.8144" width="0" layer="19" extent="1-1"/>
 </signal>
 <signal name="GND" airwireshidden="yes">
@@
 </signal>
 <signal name="VIN">
-<contactref element="AMS1117" pad="3"/>
-<contactref element="C3" pad="1"/>
-<contactref element="D1" pad="1"/>
 <contactref element="D5" pad="1"/>
 <contactref element="D2" pad="1"/>
 <contactref element="R16" pad="2"/>
-<wire x1="82.872" y1="-15.64" x2="82.85158125" y2="-16.79738125" width="0.508" layer="1"/>
-<wire x1="82.816" y1="-18.8144" x2="82.85158125" y2="-16.79738125" width="0.508" layer="1"/>
-<wire x1="84" y1="-15.64" x2="86.0886" y2="-15.64" width="0.508" layer="1"/>
-<wire x1="86.0886" y1="-15.64" x2="86.258" y2="-15.4706" width="0.508" layer="1"/>
-<wire x1="86.258" y1="-15.4706" x2="87.4" y2="-16.6126" width="0.2" layer="1"/>
 <wire x1="87.4" y1="-19.1" x2="87.7" y2="-19.4" width="0.2" layer="1"/>
 <wire x1="87.4" y1="-16.6126" x2="87.4" y2="-19.1" width="0.2" layer="1"/>
 <wire x1="95.068" y1="20.6" x2="96.267" y2="21.799" width="0.254" layer="1"/>
 <wire x1="95.068" y1="20.6" x2="89.07" y2="20.6" width="0.254" layer="1"/>
-<wire x1="82.85158125" y1="-16.79738125" x2="83.52448125" y2="-16.12448125" width="0.508" layer="1"/>
-<wire x1="83.52448125" y1="-16.12448125" x2="84" y2="-15.6489625" width="0.508" layer="1"/>
-<wire x1="84" y1="-15.6489625" x2="84" y2="-15.64" width="0.508" layer="1"/>
-<wire x1="83.3" y1="-15.64" x2="82.872" y2="-15.64" width="0.508" layer="1"/>
 <via x="83.9" y="-15.7" extent="1-16" drill="0.35"/>
-<wire x1="83.3" y1="-15.64" x2="84" y2="-15.64" width="0.508" layer="1"/>
-<wire x1="83.3" y1="-15.64" x2="83.9910375" y2="-15.64" width="0.1524" layer="1"/>
-<wire x1="83.52448125" y1="-16.12448125" x2="83.3" y2="-15.9" width="0.1524" layer="1"/>
-<wire x1="83.3" y1="-15.9" x2="83.3" y2="-15.64" width="0.1524" layer="1"/>
 <via x="89" y="20.6" extent="1-16" drill="0.35"/>
 <wire x1="89" y1="20.6" x2="89.035" y2="20.635" width="0.4064" layer="1"/>
@@
 <wire x1="84.3095" y1="17.9095" x2="87" y2="20.6" width="0.4064" layer="16"/>
 <wire x1="87" y1="20.6" x2="89" y2="20.6" width="0.4064" layer="16"/>
-<wire x1="82.872" y1="-15.64" x2="83.9910375" y2="-15.64" width="0.4064" layer="1"/>
-<wire x1="83.9910375" y1="-15.64" x2="84" y2="-15.6489625" width="0.4064" layer="1"/>
-<wire x1="82.872" y1="-15.64" x2="83.9" y2="-15.7" width="0.2" layer="1"/>
 <contactref element="R12" pad="2"/>
 <wire x1="87.7" y1="-19.4" x2="94.5" y2="-19.4" width="0.1524" layer="1"/>
@@
 <wire x1="87.9152" y1="-15.0134" x2="87.9143" y2="-15.0143" width="0.1524" layer="1"/>
 <wire x1="87.9143" y1="-15.0143" x2="87.458" y2="-15.4706" width="0.1524" layer="1"/>
-<wire x1="86.258" y1="-15.4706" x2="87.458" y2="-15.4706" width="0.1524" layer="1"/>
 <wire x1="87.9143" y1="-15.0143" x2="87.9143" y2="-9.8857" width="0.1524" layer="1"/>
 <wire x1="87.9143" y1="-9.8857" x2="88.4" y2="-9.4" width="0.1524" layer="1"/>
 <wire x1="88.4" y1="-9.4" x2="89.4848" y2="-9.4" width="0.1524" layer="1"/>
+<wire x1="87.4" y1="-16.6126" x2="87.458" y2="-15.4706" width="0" layer="19" extent="1-1"/>
+<wire x1="83.9" y1="-15.7" x2="87.458" y2="-15.4706" width="0" layer="19" extent="1-1"/>
 </signal>
 <signal name="N$25">

Commit message: schematic change
Parts:
- removed IC2: FOD817BSD, Opto-Electronic:DIP1016W60P279L460H460Q4B
- removed JP2: PINHD-2X5, Connector:2X05
- removed Q2, Q3: NMOSFET, Transistor:SOT23
- removed R12, R15, R16, R9: 10k, Resistor:RESC1608X60
- added D1: LED_BLUE, LED:LEDC1608X55N_FLAT-B
- added F1: FUSE PTC 1A, Circuit-Protection:FUSC3215X82N
- added R3, R4: 330, Resistor:RESC1608X60
- added S1, S2: (no value), Switch:B3U-1000P(M)
- added S3: DS01, Switch:DS-01
- added U4: PC817XI, SnapEDA Library:SOIC254P975X460-4N
- added X1: 057-006-1, con-panduit:057-006-1
- C11: value 0.1μ -> 100n
- C12: value 0.1µ -> 100n
- C21, C22, C6: value 100p -> 1n
- POT20: value 100K -> 10K
- R2: value 10k -> 4.7k
- R5: value 100 -> 330
- R8: value 100 -> 4.7k
- moved R8 138.9 mm to (-33.2, -53.6), turned to 0 degrees
- moved H1 66.7 mm to (33.9, -36.6)
- moved H2 65.2 mm to (48.8, -19.7)
- moved H4 28.9 mm to (42.4, -29.7)
- moved F30 4.24 mm to (16.5, -13.5)
- flipped BT2 to the bottom
Connections:
- removed net ADC_VOLTAGE_3V3: Q3.2, R9.1, U3.7
- removed net IO_RELAY_3V3: Q2.2, R15.1, U3.13
- removed net N$39: U3.33
- removed net N$40: U3.36
- removed net VIN: D2.1, D5.1, R12.2, R16.2
- new net IO_DIMMING: X1.6
- new net N$22: F1.1, PS1.5V_B, PS1.5V_T
- new net N$24: D1.A, R3.1
- new net N$27: R4.1, U4.1
- net +3.3V: no longer D4.A, Q2.1, Q3.1, R15.2, R9.2
- net 5V: now also D2.1, D4.A, D5.1, F1.2, S3.2, X1.2; no longer AMS1117.3, C3.1, JP2.2, JP2.9, PS1.5V_B, PS1.5V_T
- net ADC_CURRENT: now also X1.3; no longer JP2.7
- net ADC_VOLTAGE: now also U3.7, X1.1; no longer JP2.5, Q3.3, R12.1
- net BOOT: now also S2.1
- net DIM+: now also NEMA-7PIN.DIM-, U4.4; no longer IC2.4, JP1.6, JP2.6, NEMA-7PIN.DIM+
- net DIM-: now also NEMA-7PIN.DIM+, U4.3; no longer IC2.3, JP1.8, JP2.4, NEMA-7PIN.DIM-
- net EN: now also S1.1
- net GND: now also D1.C, K1.4, S1.2, S2.2, U4.2, X1.5; no longer IC2.2, JP2.1, JP2.10, K1.3
- net IO_RELAY: now also R8.1, U3.13, X1.4; no longer JP2.3, Q2.3, R16.1
- net N$12: now also Q1.2; no longer Q1.3
- net N$15: now also K1.3, Q1.3, R3.2; no longer K1.4, Q1.2
- net N$26: now also AMS1117.3, C3.1, S3.1; no longer IC2.1, R8.1
- net PWM_DIM: now also R4.2; no longer R8.2
- net SCL: now also U3.36
- net SDA: now also U3.33
Routing:
- net L_FUSE: track 81.0 -> 0.71 mm, vias 4 -> 1
- net VIN: track 67.0 -> 0.00 mm, vias 2 -> 0
- net N: track 57.7 -> 7.16 mm, vias 1 -> 0
- net DIM+: track 58.9 -> 9.52 mm, vias 1 -> 0
- net L: track 41.8 -> 0.00 mm, vias 1 -> 0
- net DIM-: track 44.6 -> 19.0 mm, vias 0 -> 1
- net N$23: track 18.9 -> 0.00 mm, vias 1 -> 0
- net ADC_VOLTAGE_3V3: track 17.2 -> 0.00 mm
- net L_OUT: track 15.7 -> 0.77 mm, vias 1 -> 0
- net IO_RELAY_3V3: track 14.3 -> 0.00 mm, vias 2 -> 0
- net +3.3V: track 165.4 -> 151.3 mm
- net V: track 13.1 -> 0.00 mm, vias 1 -> 0
- net 5V: track 153.7 -> 166.6 mm, vias 6 -> 5
- net N$19: track 11.6 -> 0.00 mm
- net ADC_VOLTAGE: track 69.3 -> 79.3 mm
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- removed copper zone on layer 1, net GND
Other:
- board size 148.2 x 60 mm -> 155.2 x 70 mm
