File: hardware/SMART_PJU.sch (EAGLE design)
At the start: 72 parts, among them IC1 DS3231/SO, IC10 ACS712ELCTR-05B-T, IC2 FOD817BSD, IC20 LM358_SOIC, K1 SSR, Q1 PNP, Q2 NMOSFET, Q3 NMOSFET, T20 ZMPT101B, U1 RA-01H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

Commit message: schematic change
Parts:
- removed IC2: FOD817BSD, Opto-Electronic:FOD817BSDSMT
- removed JP2: PINHD-2X5, Connector:PINHD-2X5
- removed Q2, Q3: NMOSFET, Transistor:NMOSFETSOT23-GSD
- removed R12, R15, R16, R9: 10k, Resistor:R_CHIP-0603(1608-METRIC)
- added D1: LED_BLUE, LED:CHIP-FLAT-B_0603-0.55MM
- added F1: FUSE PTC 1A, Circuit-Protection:FUSE_CHIP-1206(3216-METRIC)
- added R3, R4: 330, Resistor:R_CHIP-0603(1608-METRIC)
- added S1, S2: (no value), Switch:B3U-X000B3U-1000P(M)1000P(M)
- added S3: DS01, Switch:DS01
- added U4: PC817XI, SnapEDA Library:PC817XI
- added X1: 057-006-1, con-panduit:057-006-1
- C11: value 0.1μ -> 100n
- C12: value 0.1µ -> 100n
- C21, C22, C6: value 100p -> 1n
- POT20: value 100K -> 10K
- R2: value 10k -> 4.7k
- R5: value 100 -> 330
- R8: value 100 -> 4.7k
Connections:
- removed net ADC_VOLTAGE_3V3: Q3.S, R9.1, U3.IO35
- removed net IO_RELAY_3V3: Q2.S, R15.1, U3.IO14
- removed net N$39: U3.IO21
- removed net N$40: U3.IO22
- removed net VIN: D2.VDD, D5.VDD, R12.2, R16.2
- new net IO_DIMMING: X1-6.S
- new net N$22: F1.1, PS1.+V0
- new net N$24: D1.A, R3.1
- new net N$27: R4.1, U4.A
- net +3.3V: no longer D4.A, Q2.G, Q3.G, R15.2, R9.2
- net 5V: now also D2.VDD, D4.A, D5.VDD, F1.2, S3.2, X1-2.S; no longer AMS1117.IN, C3.1, JP2.2, JP2.9, PS1.+V0
- net ADC_CURRENT: now also X1-3.S; no longer JP2.7
- net ADC_VOLTAGE: now also U3.IO35, X1-1.S; no longer JP2.5, Q3.D, R12.1
- net BOOT: now also S2.1
- net DIM+: now also NEMA-7PIN.DIM-, U4.CT; no longer IC2.COL, JP1.6, JP2.6, NEMA-7PIN.DIM+
- net DIM-: now also NEMA-7PIN.DIM+, U4.ET; no longer IC2.EMT, JP1.8, JP2.4, NEMA-7PIN.DIM-
- net EN: now also S1.1
- net GND: now also D1.C, K1.-, S1.2, S2.2, U4.C, X1-5.S; no longer IC2.CA, JP2.1, JP2.10, K1.+
- net IO_RELAY: now also R8.1, U3.IO14, X1-4.S; no longer JP2.3, Q2.D, R16.1
- net N$12: now also Q1.E; no longer Q1.C
- net N$15: now also K1.+, Q1.C, R3.2; no longer K1.-, Q1.E
- net N$26: now also AMS1117.IN, C3.1, S3.1; no longer IC2.AN, R8.1
- net PWM_DIM: now also R4.2; no longer R8.2
- net SCL: now also U3.IO22
- net SDA: now also U3.IO21
Other:
- moved on the sheet: AMS1117, C3, C4, C5, D2, D3, D4, D5, F30, JP1, JP3, K1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
