File: hardware/Controller/JLC/controller.sch (EAGLE design)
At the start: 70 parts, among them IC1 DS3231/SO, IC10 ACS712ELCTR-05B-T, IC20 LM358_SOIC, K1 SSR, Q1 PNP, T20 ZMPT101B, U1 RA-01H, U2 AT24C64N-10SC, U3 ESP32-WROOM-32, U4 PC817XI, X1 057-006-1, X2 057-006-1

Commit message: checkpoint controller
Parts:
- removed C10, C21, C22, C6: 1n, Capacitor:C_CHIP-0603(1608-METRIC)
- removed C11, C12: 100n, Capacitor:C_CHIP-0603(1608-METRIC)
- removed C20, C23: 1µ, Capacitor:C_CHIP-0603(1608-METRIC)
- removed D1: LED_BLUE, LED:CHIP-FLAT-B_0603-0.55MM
- removed D10: 1N4448W, Diode:DIODE_1N4148W-7-F_SOD123G
- removed D3: DIODE, Diode:DIODEDO-214AC(SMA)
- removed F1: FUSE PTC 1A, Circuit-Protection:FUSE_CHIP-1206(3216-METRIC)
- removed F30: 4527, Fuse Holder:4527
- removed IC10: ACS712ELCTR-05B-T, XLKM#4:ACS712ELCTR-05B-T
- removed IC20: LM358_SOIC, IC_Linear:LM358_SOIC
- removed K1: SSR, XLKM#4:SSR
- removed NEMA-7PIN: NEMA-7P, XLKM#4:NEMA-7P
- removed POT20: 10K, Resistor:PV36W
- removed PS1: HI-LINKVERTICAL, XLKM#4:HI-LINKVERTICAL
- removed Q1: PNP, Transistor:PNP_SOT23-BEC
- removed R1, R11, R21, R23, R26, R27, R28, R29: 10k, Resistor:R_CHIP-0603(1608-METRIC)
- removed R10: 2k, Resistor:R_CHIP-0603(1608-METRIC)
- removed R2, R8: 4.7k, Resistor:R_CHIP-0603(1608-METRIC)
- removed R20: 820K, rcl:R-EU_R0805
- removed R22: 100, rcl:R-EU_R1206
- removed R24, R25: 100K, Resistor:R_CHIP-0603(1608-METRIC)
- removed R3, R4: 330, Resistor:R_CHIP-0603(1608-METRIC)
- removed T20: ZMPT101B, XLKM#4:ZMPT101B
- removed U4: PC817XI, SnapEDA Library:PC817XI
- removed V30: 10D471K, XLKM#4:VARISTOR
- removed X1: 057-006-1, con-panduit:057-006-1
- added H1, H2, H4: HOLE3.0, holes:MOUNT-HOLE3.0
Connections:
- removed net DIM+: NEMA-7PIN.DIM-, U4.CT
- removed net DIM-: NEMA-7PIN.DIM+, U4.ET
- removed net L: F30.1, NEMA-7PIN.L
- removed net L_FUSE: F30.2, IC10.IP+, PS1.AC_1, R20.2, V30.1
- removed net L_OUT: IC10.IP-, K1.L1
- removed net L_ZMPT: R20.1, T20.1
- removed net N: NEMA-7PIN.N, PS1.AC_2, T20.2, V30.2
- removed net N$1: C20.1, R22.1, T20.3
- removed net N$11: C10.1, IC10.FILTER
- removed net N$12: D3.C, Q1.E, R2.2
- removed net N$13: Q1.B, R1.1, R2.1
- removed net N$15: K1.+, Q1.C, R3.2
- removed net N$16: C22.2, IC20.-IN2, R21.2, R25.1
- removed net N$17: C23.2, R21.1
- removed net N$18: C23.1, POT20.P$2
- removed net N$2: C21.2, IC20.OUT1
- removed net N$22: F1.1, PS1.+V0
- removed net N$24: D1.A, R3.1
- removed net N$27: R4.1, U4.A
- removed net N$3: C20.2, R23.1
- removed net N$4: IC10.VIOUT, R10.1
- removed net N$7: C22.1, IC20.OUT2
- removed net N$8: C21.1, IC20.-IN1, R23.2, R24.1
- removed net N$9: D10.A, R10.2, R11.2
- removed net OUT-A: POT20.P$1, R24.2
- removed net POS-A: IC20.+IN1, R22.2, R26.1, R27.2, T20.4
- removed net POS-B: IC20.+IN2, R28.1, R29.2
- removed net V: K1.L2, NEMA-7PIN.V
- net 5V: no longer C11.1, C6.2, D3.A, F1.2, IC10.VCC, IC20.V+, R26.2, R28.2, X1-2.S
- net ADC_CURRENT: no longer C12.1, D10.C, X1-3.S
- net ADC_VOLTAGE: no longer R25.2, X1-1.S
- net GND: no longer C10.2, C11.2, C12.2, C6.1, D1.C, IC10.GND, IC20.V-, K1.-, POT20.P$3, PS1.-V0, R11.1, R27.1, R29.1, U4.C, X1-5.S
- net IO_DIMMING: no longer X1-6.S
- net IO_RELAY: no longer R1.2, R8.1, X1-4.S
- net PWM_DIM: no longer R4.2
