File: hardware/Power/Single Layer/power.brd (EAGLE design)
At the start: 71 x 71 mm, 42 parts, among them IC1 ACS712ELCTR-05B-T, IC2 LM358_SOIC, Q1 PNP, T1 ZMPT101B, X1 057-006-1

Commit message: feat : checkpoint 2
Parts:
- added JP1, JP2: 330, Resistor:RESC2012X65
- moved R13 1.90 mm to (-28.9, 0.85)
- moved R14 1.06 mm to (-28.8, -1.93)
- moved C2 0.70 mm to (-25.0, -1.93)
- moved C8 0.70 mm to (-16.1, -2.08)
- moved R15 0.70 mm to (-21.2, -1.82)
Connections:
- net 5V: now also JP1.1, JP1.2
- net POS-B: now also JP2.1, JP2.2
Routing:
- net POS-B: track 9.15 -> 8.38 mm, vias 2 -> 0
- net N$16: track 14.0 -> 14.7 mm
- net N$18: track 12.2 -> 12.9 mm
- net 5V: track 123.6 -> 123.8 mm, vias 4 -> 2
