File: hardware/Controller/controller.sch (EAGLE design)
At the start: 29 parts, among them IC1 DS3231/SO, IC2 AT24C64N-10SC, U1 NCP1117ST33T3G, X2 057-006-1

Commit message: bakcup before ganti ukuran smd
Parts:
- added PH1: LDR, photo-elements:A1050_09
- added R4: 10K, Resistor:R_CHIP-0603(1608-METRIC)
- C1, C2, C3, C4: device Capacitor:C_CHIP-0603(1608-METRIC) -> Capacitor:C_CHIP-0805(2012-METRIC)
- LED: device LED:CHIP-FLAT-B_0603-0.55MM -> LED:CHIP-FLAT-B_0805
- R1, R2, R3, R5, R6: device Resistor:R_CHIP-0603(1608-METRIC) -> Resistor:R_CHIP-0805(2012-METRIC)
- renumbered U1 to REG-3V3
Connections:
- removed net N$10: IC2.A2, RN2C.1
- removed net N$26: C3.1, REG-3V3.IN, S3.1
- removed net N$33: REG-3V3.GND
- removed net N$5: IC2.A0, RN2A.1
- removed net N$6: IC2.A1, RN2B.1
- new net 5V_IN: NEO1.VDD, NEO2.VDD, S3.2, X2-2.S
- new net A0: IC2.A0, RN1A.2
- new net A1: IC2.A1, RN2D.2
- new net A2: IC2.A2, RN2C.2
- new net ADC_LIGHT: ESP32.SENSOR_VP, PH1.1, R4.1
- net +3.3V: now also R4.2, RN2A.1, RN2B.1, RN2C.1, RN2D.1; no longer RN1D.1, RN2A.2, RN2B.2, RN2C.2
- net 5V: now also C3.1, REG-3V3.IN, S3.1; no longer NEO1.VDD, NEO2.VDD, S3.2, X2-2.S
- net GND: now also PH1.2, REG-3V3.GND
- net N$21: now also RN1C.2; no longer RN1A.2
- net SCL: now also RN2A.2; no longer RN1C.2
- net SDA: now also RN2B.2; no longer RN1D.2
Other:
- moved on the sheet: BT, C1, C2, IC1, IC2, LED, NEO1, NEO2, R1, RN1A, RN1B, RN1C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

Commit message: checkpoint sebelum cetak single layer
Parts:
- removed BT: (no value), SparkFun-Batteries:BATTERY-20MM_PTH
- removed C1: 100n, Capacitor:C_CHIP-0805(2012-METRIC)
- removed C2: 1μ, Capacitor:C_CHIP-0805(2012-METRIC)
- removed H1, H2, H3: HOLE3.0, holes:MOUNT-HOLE3.0
- removed IC1: DS3231/SO, XLKM#4:DS3231/SO
- removed IC2: AT24C64N-10SC, XLKM#4:AT24C64N-10SC
- removed RN1, RN2: (no value), resistor-dil:4R-NCAY16
- removed X2: 057-006-1, con-panduit:057-006-1
- added U$1: DS3231_MODULE, XLKM#4:DS3231_MODULE
- added X1: 057-006-1, con-panduit:057-006-1
Connections:
- removed net A0: IC2.A0, RN1A.2
- removed net A1: IC2.A1, RN2D.2
- removed net A2: IC2.A2, RN2C.2
- removed net N$19: BT.+, IC1.VBAT
- removed net N$20: IC1.SQW/INT, RN1B.2
- removed net N$21: IC1.32KHZ, RN1C.2
- removed net N$23: BT.-, C1.2
- removed net N$41: ESP32.IO23
- removed net N$43: ESP32.IO26
- removed net N$44: ESP32.IO27
- new net --: U$1.VCC
- new net -1: ESP32.IO21
- new net -2: ESP32.IO19
- new net -3: ESP32.IO12
- net +3.3V: now also U$1.VCC2; no longer C1.1, C2.1, IC1.VCC, IC2.VCC, RN1A.1, RN1B.1, RN1C.1, RN2A.1, RN2B.1, RN2C.1, RN2D.1
- net 5V_IN: now also X1-2.S; no longer X2-2.S
- net ADC_CURRENT: now also X1-4.S; no longer X2-3.S
- net ADC_VOLTAGE: now also X1-1.S; no longer X2-1.S
- net GND: now also U$1.GND, U$1.GND2, X1-6.S; no longer C2.2, IC1.GND, IC2.GND, IC2.WP, X2-5.S
- net IO_DIMMING: now also ESP32.IO27, X1-5.S; no longer ESP32.IO12, X2-6.S
- net IO_RELAY: now also ESP32.IO26, X1-3.S; no longer ESP32.IO14, X2-4.S
- net LED: now also ESP32.IO14; no longer ESP32.IO19
- net SCL: now also U$1.SCL; no longer IC1.SCL, IC2.SCL, RN2A.2
- net SDA: now also ESP32.IO23, U$1.SDA; no longer ESP32.IO21, IC1.SDA, IC2.SDA, RN2B.2

Commit message: checkpoint 21/05
Connections:
- net 5V_IN: now also X1-1.S; no longer X1-2.S
- net ADC_CURRENT: now also X1-3.S; no longer X1-4.S
- net ADC_VOLTAGE: now also X1-2.S; no longer X1-1.S
- net GND: now also X1-5.S; no longer X1-6.S
- net IO_DIMMING: now also X1-6.S; no longer X1-5.S
- net IO_RELAY: now also X1-4.S; no longer X1-3.S
Other:
- moved on the sheet: X1-3, X1-4, X1-5, X1-6
Changed lines of the file:
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@@
 <attribute name="NAME" x="-128.016" y="-32.258" size="1.524" layer="95" rot="R180"/>
 </instance>
-<instance part="X1" gate="-4" x="-139.7" y="-38.1" smashed="yes">
+<instance part="X1" gate="-3" x="-139.7" y="-38.1" smashed="yes">
 <attribute name="NAME" x="-138.684" y="-38.862" size="1.524" layer="95"/>
 </instance>
-<instance part="X1" gate="-3" x="-127" y="-38.1" smashed="yes" rot="R180">
+<instance part="X1" gate="-4" x="-127" y="-38.1" smashed="yes" rot="R180">
 <attribute name="NAME" x="-128.016" y="-37.338" size="1.524" layer="95" rot="R180"/>
 </instance>
-<instance part="X1" gate="-6" x="-139.7" y="-43.18" smashed="yes">
+<instance part="X1" gate="-5" x="-139.7" y="-43.18" smashed="yes">
 <attribute name="NAME" x="-138.684" y="-43.942" size="1.524" layer="95"/>
 </instance>
-<instance part="X1" gate="-5" x="-127" y="-43.18" smashed="yes" rot="R180">
+<instance part="X1" gate="-6" x="-127" y="-43.18" smashed="yes" rot="R180">
 <attribute name="NAME" x="-128.016" y="-42.418" size="1.524" layer="95" rot="R180"/>
 </instance>
@@
 </segment>
 <segment>
-<pinref part="X1" gate="-6" pin="S"/>
+<pinref part="X1" gate="-5" pin="S"/>
 <wire x1="-144.78" y1="-43.18" x2="-147.32" y2="-43.18" width="0.1524" layer="91"/>
 <label x="-147.32" y="-43.18" size="1.778" layer="95" rot="R180" xref="yes"/>
@@
 </segment>
 <segment>
-<pinref part="X1" gate="-4" pin="S"/>
+<pinref part="X1" gate="-3" pin="S"/>
 <wire x1="-144.78" y1="-38.1" x2="-147.32" y2="-38.1" width="0.1524" layer="91"/>
 <label x="-147.32" y="-38.1" size="1.778" layer="95" rot="R180" xref="yes"/>
@@
 </segment>
 <segment>
-<pinref part="X1" gate="-1" pin="S"/>
-<wire x1="-144.78" y1="-33.02" x2="-147.32" y2="-33.02" width="0.1524" layer="91"/>
-<label x="-147.32" y="-33.02" size="1.778" layer="95" rot="R180" xref="yes"/>
+<pinref part="X1" gate="-2" pin="S"/>
+<wire x1="-121.92" y1="-33.02" x2="-119.38" y2="-33.02" width="0.1524" layer="91"/>
+<label x="-119.38" y="-33.02" size="1.778" layer="95" xref="yes"/>
 </segment>
 </net>
@@
 <net name="IO_RELAY" class="0">
 <segment>
-<pinref part="X1" gate="-3" pin="S"/>
+<pinref part="X1" gate="-4" pin="S"/>
 <wire x1="-121.92" y1="-38.1" x2="-119.38" y2="-38.1" width="0.1524" layer="91"/>
 <label x="-119.38" y="-38.1" size="1.778" layer="95" xref="yes"/>
@@
 <net name="IO_DIMMING" class="0">
 <segment>
-<pinref part="X1" gate="-5" pin="S"/>
+<pinref part="X1" gate="-6" pin="S"/>
 <wire x1="-121.92" y1="-43.18" x2="-119.38" y2="-43.18" width="0.1524" layer="91"/>
 <label x="-119.38" y="-43.18" size="1.778" layer="95" xref="yes"/>
@@
 </segment>
 <segment>
-<pinref part="X1" gate="-2" pin="S"/>
-<wire x1="-121.92" y1="-33.02" x2="-119.38" y2="-33.02" width="0.1524" layer="91"/>
-<label x="-119.38" y="-33.02" size="1.778" layer="95" xref="yes"/>
-</segment>
-</net>
+<pinref part="X1" gate="-1" pin="S"/>
+<wire x1="-144.78" y1="-33.02" x2="-147.32" y2="-33.02" width="0.1524" layer="91"/>
+<label x="-147.32" y="-33.02" size="1.778" layer="95" rot="R180" xref="yes"/>
+</segment>
+</net>
