File: hardware/Controller/controller.sch (EAGLE design)
At the start: 22 parts, among them X1 057-006-1

Commit message: feat : checkpoint for interface dev 👾
Connections:
- net 5V_IN: now also X1-2.S; no longer X1-1.S
- net ADC_CURRENT: now also X1-4.S; no longer X1-3.S
- net ADC_VOLTAGE: now also X1-1.S; no longer X1-2.S
- net GND: now also X1-6.S; no longer X1-5.S
- net IO_DIMMING: now also X1-5.S; no longer X1-6.S
- net IO_RELAY: now also X1-3.S; no longer X1-4.S
Other:
- moved on the sheet: X1-3, X1-4, X1-5, X1-6
Changed lines of the file:
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@@
 <attribute name="NAME" x="-128.016" y="-32.258" size="1.524" layer="95" rot="R180"/>
 </instance>
-<instance part="X1" gate="-3" x="-139.7" y="-38.1" smashed="yes">
+<instance part="X1" gate="-4" x="-139.7" y="-38.1" smashed="yes">
 <attribute name="NAME" x="-138.684" y="-38.862" size="1.524" layer="95"/>
 </instance>
-<instance part="X1" gate="-4" x="-127" y="-38.1" smashed="yes" rot="R180">
+<instance part="X1" gate="-3" x="-127" y="-38.1" smashed="yes" rot="R180">
 <attribute name="NAME" x="-128.016" y="-37.338" size="1.524" layer="95" rot="R180"/>
 </instance>
-<instance part="X1" gate="-5" x="-139.7" y="-43.18" smashed="yes">
+<instance part="X1" gate="-6" x="-139.7" y="-43.18" smashed="yes">
 <attribute name="NAME" x="-138.684" y="-43.942" size="1.524" layer="95"/>
 </instance>
-<instance part="X1" gate="-6" x="-127" y="-43.18" smashed="yes" rot="R180">
+<instance part="X1" gate="-5" x="-127" y="-43.18" smashed="yes" rot="R180">
 <attribute name="NAME" x="-128.016" y="-42.418" size="1.524" layer="95" rot="R180"/>
 </instance>
@@
 </segment>
 <segment>
-<pinref part="X1" gate="-5" pin="S"/>
+<pinref part="X1" gate="-6" pin="S"/>
 <wire x1="-144.78" y1="-43.18" x2="-147.32" y2="-43.18" width="0.1524" layer="91"/>
 <label x="-147.32" y="-43.18" size="1.778" layer="95" rot="R180" xref="yes"/>
@@
 </segment>
 <segment>
-<pinref part="X1" gate="-3" pin="S"/>
+<pinref part="X1" gate="-4" pin="S"/>
 <wire x1="-144.78" y1="-38.1" x2="-147.32" y2="-38.1" width="0.1524" layer="91"/>
 <label x="-147.32" y="-38.1" size="1.778" layer="95" rot="R180" xref="yes"/>
@@
 </segment>
 <segment>
-<pinref part="X1" gate="-2" pin="S"/>
-<wire x1="-121.92" y1="-33.02" x2="-119.38" y2="-33.02" width="0.1524" layer="91"/>
-<label x="-119.38" y="-33.02" size="1.778" layer="95" xref="yes"/>
+<pinref part="X1" gate="-1" pin="S"/>
+<wire x1="-144.78" y1="-33.02" x2="-147.32" y2="-33.02" width="0.1524" layer="91"/>
+<label x="-147.32" y="-33.02" size="1.778" layer="95" rot="R180" xref="yes"/>
 </segment>
 </net>
@@
 <net name="IO_RELAY" class="0">
 <segment>
-<pinref part="X1" gate="-4" pin="S"/>
+<pinref part="X1" gate="-3" pin="S"/>
 <wire x1="-121.92" y1="-38.1" x2="-119.38" y2="-38.1" width="0.1524" layer="91"/>
 <label x="-119.38" y="-38.1" size="1.778" layer="95" xref="yes"/>
@@
 <net name="IO_DIMMING" class="0">
 <segment>
-<pinref part="X1" gate="-6" pin="S"/>
+<pinref part="X1" gate="-5" pin="S"/>
 <wire x1="-121.92" y1="-43.18" x2="-119.38" y2="-43.18" width="0.1524" layer="91"/>
 <label x="-119.38" y="-43.18" size="1.778" layer="95" xref="yes"/>
@@
 </segment>
 <segment>
-<pinref part="X1" gate="-1" pin="S"/>
-<wire x1="-144.78" y1="-33.02" x2="-147.32" y2="-33.02" width="0.1524" layer="91"/>
-<label x="-147.32" y="-33.02" size="1.778" layer="95" rot="R180" xref="yes"/>
-</segment>
-</net>
+<pinref part="X1" gate="-2" pin="S"/>
+<wire x1="-121.92" y1="-33.02" x2="-119.38" y2="-33.02" width="0.1524" layer="91"/>
+<label x="-119.38" y="-33.02" size="1.778" layer="95" xref="yes"/>
+</segment>
+</net>
