File: hardware/Controller/controller.brd (EAGLE design)
At the start: 66 x 66 mm, 29 parts, among them IC1 DS3231/SO, IC2 AT24C64N-10SC, U1 NCP1117ST33T3G, X2 057-006-1

Commit message: bakcup before ganti ukuran smd
Parts:
- removed U1: NCP1117ST33T3G, IC_Power-Management:SOT230P700X170-4
- added PH1: LDR, photo-elements:T0-46-A10XX
- added R4: 10K, Resistor:RESC1608X60
- added REG-3V3: NCP1117ST33T3G, IC_Power-Management:SOT230P700X170-4
- C1, C2, C3, C4: device Capacitor:CAPC1608X85 -> Capacitor:CAPC2012X110
- LED: device LED:LEDC1608X55N_FLAT-B -> LED:LEDC2012X110N_FLAT-B
- R1, R2, R3, R5, R6: device Resistor:RESC1608X60 -> Resistor:RESC2012X65
- moved H3 83.4 mm to (-18.0, 21.4)
- moved R2 61.9 mm to (-0.32, -9.56), turned to 270 degrees
- moved R3 60.6 mm to (-0.29, -5.82), turned to 270 degrees
- moved X2 47.2 mm to (0.00, -24.1)
- moved H2 32.8 mm to (28.5, 2.60)
- moved H1 30.6 mm to (-19.7, -18.8)
- moved S3 25.4 mm to (-10.9, -23.2), turned to 180 degrees
- moved IC2 17.7 mm to (20.9, -8.55), flipped to the top
- moved NEO1 17.3 mm to (11.6, -16.9)
- moved NEO2 16.2 mm to (19.8, -17.0)
- moved R1 11.3 mm to (-3.73, -5.72), turned to 90 degrees
- moved EN 10.2 mm to (3.01, 25.0), turned to 90 degrees
- moved C1 8.98 mm to (5.28, 14.7), turned to 270 degrees
- moved RN1 8.31 mm to (10.2, -6.83), turned to 180 degrees
- moved LED 8.08 mm to (-3.78, -9.82), turned to 270 degrees
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Connections:
- removed net N$10: IC2.3, RN2.3
- removed net N$26: C3.1, S3.1, U1.3
- removed net N$33: U1.1
- removed net N$5: IC2.1, RN2.1
- removed net N$6: IC2.2, RN2.2
- new net 5V_IN: NEO1.1, NEO2.1, S3.2, X2.2
- new net A0: IC2.1, RN1.8
- new net A1: IC2.2, RN2.5
- new net A2: IC2.3, RN2.6
- new net ADC_LIGHT: ESP32.4, PH1.1, R4.1
- net +3.3V: now also R4.2, REG-3V3.2, RN2.1, RN2.2, RN2.3, RN2.4; no longer RN1.4, RN2.6, RN2.7, RN2.8, U1.2
- net 5V: now also C3.1, REG-3V3.3, S3.1; no longer NEO1.1, NEO2.1, S3.2, X2.2
- net GND: now also PH1.2, REG-3V3.1
- net N$21: now also RN1.6; no longer RN1.8
- net SCL: now also RN2.8; no longer RN1.6
- net SDA: now also RN2.7; no longer RN1.5
Routing:
- net IO_RELAY: track 0.04 -> 30.0 mm
- net ADC_CURRENT: track 0.00 -> 29.6 mm
- net +3.3V: track 117.2 -> 90.3 mm, vias 5 -> 0
- net EN: track 23.7 -> 0.00 mm, vias 1 -> 0
- net IO_DIMMING: track 0.00 -> 19.0 mm
- net N$2: track 0.00 -> 17.7 mm
- net 5V_IN: track 0.00 -> 14.3 mm
- net 5V: track 0.01 -> 13.9 mm
- net ADC_VOLTAGE: track 0.00 -> 13.5 mm
- net A2: track 0.00 -> 11.0 mm
- net A0: track 0.00 -> 10.9 mm
- net A1: track 0.00 -> 10.6 mm
- net SCL: track 19.0 -> 9.95 mm
- net SDA: track 19.0 -> 12.8 mm
- net LED: track 5.89 -> 0.14 mm
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- removed copper zone on layer 16, net GND

Commit message: checkpoint sebelum cetak single layer
Parts:
- removed BT: (no value), SparkFun-Batteries:BATTCOM_20MM_PTH
- removed C1: 100n, Capacitor:CAPC2012X110
- removed C2: 1μ, Capacitor:CAPC2012X110
- removed H1, H2, H3: HOLE3.0, holes:3,0
- removed IC1: DS3231/SO, XLKM#4:SO16W
- removed IC2: AT24C64N-10SC, XLKM#4:SOIC127P600X175-8N
- removed RN1, RN2: (no value), resistor-dil:CAY16
- removed X2: 057-006-1, con-panduit:057-006-1
- added U$1: DS3231_MODULE, XLKM#4:DS3231_MODULE
- added X1: 057-006-1, con-panduit:057-006-1
- moved R6 38.0 mm to (5.61, 26.9), turned to 180 degrees
- moved R5 10.1 mm to (5.63, 24.5), turned to 0 degrees
- moved NEO2 9.44 mm to (20.2, -7.56)
- moved NEO1 9.33 mm to (12.3, -7.56)
- moved BOOT 7.68 mm to (2.10, 25.8)
- moved R4 6.61 mm to (-22.4, -6.50), turned to 90 degrees
- moved EN 6.13 mm to (9.11, 25.6), turned to 270 degrees
- moved R2 3.72 mm to (3.15, -10.9)
- moved R3 3.72 mm to (3.17, -7.18)
- moved PH1 3.44 mm to (-22.9, -12.7), turned to 180 degrees
- moved R1 2.86 mm to (-1.18, -7.02)
- moved LED 2.86 mm to (-1.23, -11.1)
- moved REG-3V3 2.86 mm to (-7.39, -9.25)
- moved C6 2.86 mm to (-17.0, -7.39)
- moved C3 2.84 mm to (-5.07, -16.1)
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Connections:
- removed net A0: IC2.1, RN1.8
- removed net A1: IC2.2, RN2.5
- removed net A2: IC2.3, RN2.6
- removed net N$19: BT.1, IC1.14
- removed net N$20: IC1.3, RN1.7
- removed net N$21: IC1.1, RN1.6
- removed net N$23: BT.2, C1.2
- removed net N$41: ESP32.37
- removed net N$43: ESP32.11
- removed net N$44: ESP32.12
- new net --: U$1.VCC
- new net -1: ESP32.33
- new net -2: ESP32.31
- new net -3: ESP32.14
- net +3.3V: now also U$1.VCC2; no longer C1.1, C2.1, IC1.2, IC2.8, RN1.1, RN1.2, RN1.3, RN2.1, RN2.2, RN2.3, RN2.4
- net 5V_IN: now also X1.2; no longer X2.2
- net ADC_CURRENT: now also X1.4; no longer X2.3
- net ADC_VOLTAGE: now also X1.1; no longer X2.1
- net GND: now also U$1.GND, U$1.GND2, X1.6; no longer C2.2, IC1.13, IC2.4, IC2.7, X2.5
- net IO_DIMMING: now also ESP32.12, X1.5; no longer ESP32.14, X2.6
- net IO_RELAY: now also ESP32.11, X1.3; no longer ESP32.13, X2.4
- net LED: now also ESP32.13; no longer ESP32.31
- net SCL: now also U$1.SCL; no longer IC1.16, IC2.6, RN2.8
- net SDA: now also ESP32.37, U$1.SDA; no longer ESP32.33, IC1.15, IC2.5, RN2.7
Routing:
- net EN: track 0.00 -> 75.3 mm, vias 0 -> 2
- net +3.3V: track 90.3 -> 140.4 mm, vias 0 -> 2
- net 5V_IN: track 14.3 -> 64.1 mm
- net BOOT: track 0.97 -> 34.5 mm, vias 0 -> 2
- net ADC_LIGHT: track 0.00 -> 26.7 mm, vias 0 -> 1
- net TX0: track 0.00 -> 24.5 mm, vias 0 -> 2
- net ANT: track 0.00 -> 19.5 mm, vias 0 -> 1
- net LED: track 0.14 -> 16.2 mm
- net IO_DIMMING: track 19.0 -> 31.4 mm
- net A2: track 11.0 -> 0.00 mm
- net A0: track 10.9 -> 0.00 mm
- net A1: track 10.6 -> 0.00 mm
- net RX0: track 0.00 -> 9.90 mm
- net SDA: track 12.8 -> 4.04 mm
- net SCL: track 9.95 -> 3.52 mm
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- added copper zone on layer 1, net GND
- added copper zone on layer 16, net GND
Other:
- board text added: "Controller Board"
- board text added: "V2"

Commit message: checkpoint 21/05
Parts:
- moved X1 0.10 mm to (0.00, -23.8), flipped to the bottom, turned to 180 degrees
Connections:
- net 5V_IN: now also X1.1; no longer X1.2
- net ADC_CURRENT: now also X1.3; no longer X1.4
- net ADC_VOLTAGE: now also X1.2; no longer X1.1
- net GND: now also X1.5; no longer X1.6
- net IO_DIMMING: now also X1.6; no longer X1.5
- net IO_RELAY: now also X1.4; no longer X1.3
Other:
- board text added: "ANT"

Commit message: feat : react to esp32 script
Parts:
- BOOT, EN: value (none) -> SWITCH; device Switch:B3U-1000P(M) -> XLKM#4:SW_1437566-3
- moved EN 6.46 mm to (3.98, 29.6), turned to 0 degrees
- moved R6 5.98 mm to (-0.35, 26.5), turned to 0 degrees
- moved R5 3.33 mm to (8.31, 26.4), turned to 180 degrees
- moved BOOT 3.18 mm to (4.05, 23.3), turned to 0 degrees
- moved JP1 2.72 mm to (-8.24, 25.1)
Routing:
- net EN: track 75.3 -> 64.5 mm
- net BOOT: track 34.5 -> 42.2 mm
- net +3.3V: track 140.8 -> 139.2 mm, vias 2 -> 0
- net NSS: track 18.7 -> 17.9 mm
- net MOSI: track 23.2 -> 22.6 mm
Other:
- board text added: "V2.5"
- board text removed: "V2"

Commit message: feat : checkpoint for interface dev 👾
Connections:
- net 5V_IN: now also X1.2; no longer X1.1
- net ADC_CURRENT: now also X1.4; no longer X1.3
- net ADC_VOLTAGE: now also X1.1; no longer X1.2
- net GND: now also X1.6; no longer X1.5
- net IO_DIMMING: now also X1.5; no longer X1.6
- net IO_RELAY: now also X1.3; no longer X1.4
Routing:
- net ADC_CURRENT: track 29.3 -> 32.9 mm
- net IO_RELAY: track 33.4 -> 30.0 mm
- net ADC_VOLTAGE: track 18.1 -> 15.5 mm
- net 5V_IN: track 63.6 -> 61.1 mm
- net IO_DIMMING: track 31.5 -> 29.1 mm
